Commit message: URDF with battery holder + Lower COM at high speed

File: 05-simulation/felin/felin.urdf (robot description, URDF)
Before this commit: robot felin, 17 links, 16 joints
Links:
- link FL-femur: mass 0.05 -> 0.5
- link FL-tibia: mass 0.05 -> 0.1
- link FR-femur: mass 0.05 -> 0.5
- link FR-tibia: mass 0.05 -> 0.1
- link RL-femur: mass 0.05 -> 0.5
- link RL-tibia: mass 0.05 -> 0.1
- link RR-femur: mass 0.05 -> 0.5
- link RR-tibia: mass 0.05 -> 0.1
- link body-base: mass 3 -> 3.0; geometry collision box size=0.178 0.060 0.028; collision box size=0.220 0.120 0.080

Commit message: up

File: 05-simulation/felin/felin.urdf (robot description, URDF)
Before this commit: robot felin, 17 links, 16 joints
Links:
- link body-base: mass 2.6 -> 2.4
