Commit message: up

File: 02-kinematics/felin.urdf (robot description, URDF)
Before this commit: robot felin, 17 links, 16 joints
Links:
- link FL-pod: mass 0.5 -> 0.4
- link FR-pod: mass 0.5 -> 0.4
- link RL-pod: mass 0.5 -> 0.4
- link RR-pod: mass 0.5 -> 0.4
- link body-base: mass 3.0 -> 2.6

Commit message: crouch improvement

File: 02-kinematics/felin.urdf (robot description, URDF)
Before this commit: robot felin, 17 links, 16 joints
Links:
- link FL-femur: geometry collision box size=0.140 0.054 0.040; collision cylinder length=0.040 radius=0.027
- link FR-femur: geometry collision box size=0.140 0.054 0.040; collision cylinder length=0.040 radius=0.027
- link RL-femur: geometry collision box size=0.140 0.054 0.040; collision cylinder length=0.040 radius=0.027
- link RR-femur: geometry collision box size=0.140 0.054 0.040; collision cylinder length=0.040 radius=0.027

File: 05-simulation/felin/felin.urdf (robot description, URDF)
Before this commit: robot felin, 17 links, 16 joints
Links:
- link FL-femur: geometry collision box size=0.140 0.054 0.040; collision cylinder length=0.040 radius=0.027
- link FR-femur: geometry collision box size=0.140 0.054 0.040; collision cylinder length=0.040 radius=0.027
- link RL-femur: geometry collision box size=0.140 0.054 0.040; collision cylinder length=0.040 radius=0.027
- link RR-femur: geometry collision box size=0.140 0.054 0.040; collision cylinder length=0.040 radius=0.027
- link body-base: mass 2.4 -> 2.6

File: 06-firmware/felin/felin.urdf (robot description, URDF)
Before this commit: robot felin, 17 links, 16 joints
Links:
- link FL-femur: geometry collision box size=0.140 0.054 0.040; collision cylinder length=0.040 radius=0.027
- link FR-femur: geometry collision box size=0.140 0.054 0.040; collision cylinder length=0.040 radius=0.027
- link RL-femur: geometry collision box size=0.140 0.054 0.040; collision cylinder length=0.040 radius=0.027
- link RR-femur: geometry collision box size=0.140 0.054 0.040; collision cylinder length=0.040 radius=0.027
- link body-base: mass 2.4 -> 2.6
